File: project/fpga.kicad_sch (KiCad schematic)
At the start: 0 parts

Commit message: Inicio de la PCB y conexion del PLL
Parts:
- added U6: ICE40HX4K-TQ144, Package_QFP:TQFP-144_20x20mm_P0.5mm, symbol FPGA_Lattice:ICE40HX4K-TQ144
Connections:
- new net: U6.30 (VCCIO_3), U6.6 (VCCIO_3)
- new net: U6.46 (VCCIO_2), U6.57 (VCCIO_2)
- new net: U6.100 (VCCIO_1), U6.89 (VCCIO_1)
- new net: U6.123 (VCCIO_0), U6.131 (VCCIO_0)
- new net VUART_CTS: U6.61 (IOB_96)
- new net VUART_DCD: U6.64 (IOB_104_CBSEL1)
- new net VUART_DSR: U6.63 (IOB_103_CBSEL0)
- new net VUART_DTR: U6.62 (IOB_102)
- new net VUART_RTS: U6.60 (IOB_95)
- new net VUART_Rx: U6.55 (IOB_91)
- new net VUART_Tx: U6.56 (IOB_94)
- no-connect marks 0 -> 11
