File: project/perifericos.kicad_sch (KiCad schematic)
At the start: 68 parts, among them P1 Conector SMD 2x10, P2 Conector SMD 2x10, P3 Conector SMD 2x10, P4 Conector SMD 2x10, SW1 SW_Push, SW2 SW_Push, SW3 SW_Push, SW4 SW_Push, SW5 SW_Push, SW6 SW_Push, SW7 SW_Push, SW8 SW_Push, U6 ICE40HX4K-TQ144, Y2 ECS-3225MVQ-1000-CN-TR

Commit message: - Included properties such as Reference, Value, Footprint, and various manufacturer details. - Defined 20 pins with appropriate names and attributes for the symbol. - Ensured compatibility with KiCad version 8.0 and above.
Parts:
- C34, C35, C36, C37, C38, C39, C40, C41, C43, C44, C45, C46, C47, C48, C49, C50, C51, C52, C53, C54: footprint (none) -> Capacitor_SMD:C_1206_3216Metric
- P1, P2, P3, P4: footprint (none) -> FRT-FPGA:Header 2x10 SMD
- R25, R26, R27, R28, R29, R30, R31, R32, R33, R34, R35, R36, R37, R38, R39, R40, R41, R42, R43, R44, R45, R46, R47, R48: footprint (none) -> Resistor_SMD:R_1206_3216Metric
- Y2: footprint ECS3225MVQ1000CNTR -> ECS_3225MV_120_CN_TR:OSC_ECS-3225MV-120-CN-TR
