File: project/perifericos.kicad_sch (KiCad schematic)
At the start: 68 parts, among them P1 Conector 2x10, P2 Conector 2x10, P3 Conector 2x10, P4 Conector 2x10, SW1 SW_Push, SW2 SW_Push, SW3 SW_Push, SW4 SW_Push, SW5 SW_Push, SW6 SW_Push, SW7 SW_Push, SW8 SW_Push, U6 ICE40HX4K-TQ144, Y2 ECS-3225MVQ-1000-CN-TR

Commit message: cambio a nombre final, agregado de licencia en esquematico y etiqueta
Other:
- company: (none) -> Maximiliano Simonazzi, Valentin Gomez Espeche
- title: (none) -> Azukar FPGA

Commit message: Version 2 de pcb completa, falta revisar silkscreen y ajustes menores
Parts:
- added JP2: SolderJumper_2_Open, Jumper:SolderJumper-2_P1.3mm_Open_TrianglePad1.0x1.5mm, symbol Jumper:SolderJumper_2_Open
- renumbered C42 to C33, C43 to C34, C44 to C35, C45 to C36, C46 to C37, C47 to C38, C48 to C39, C49 to C40, C50 to C41, C51 to C42, C52 to C43, C53 to C44, C54 to C45, C34 to C46, C35 to C47, C36 to C48, C37 to C49, C38 to C50, C39 to C51, C40 to C52, C41 to C53, D11 to D10, D12 to D11, D5 to D4, D6 to D5, D7 to D6, D8 to D7, D9 to D8, D10 to D9, P3 to P1, P1 to P2, P2 to P3
Connections:
- net BOT1: now also U6.110 (IOT_168); no longer U6.37 (IOB_56)
- net BOT2: now also U6.112 (IOT_169); no longer U6.38 (IOB_57)
- net BOT3: now also U6.113 (IOT_170); no longer U6.39 (IOB_61)
- net BOT4: now also U6.114 (IOT_171); no longer U6.41 (IOB_63)
- net BOT5: now also U6.115 (IOT_172); no longer U6.42 (IOB_64)
- net BOT6: now also U6.116 (IOT_173); no longer U6.43 (IOB_71)
- net BOT7: now also U6.117 (IOT_174); no longer U6.44 (IOB_72)
- net BOT8: now also U6.118 (IOT_177); no longer U6.45 (IOB_73)
- net LED1: now also U6.37 (IOB_56); no longer U6.110 (IOT_168)
- net LED2: now also U6.38 (IOB_57); no longer U6.112 (IOT_169)
- net LED3: now also U6.39 (IOB_61); no longer U6.113 (IOT_170)
- net LED4: now also U6.41 (IOB_63); no longer U6.114 (IOT_171)
- net LED5: now also U6.42 (IOB_64); no longer U6.115 (IOT_172)
- net LED6: now also U6.43 (IOB_71); no longer U6.116 (IOT_173)
- net LED7: now also U6.44 (IOB_72); no longer U6.117 (IOT_174)
- net LED8: now also U6.45 (IOB_73); no longer U6.118 (IOT_177)
- net VUART_DCD: now also U6.55 (IOB_91); no longer U6.64 (IOB_104_CBSEL1)
- net VUART_DSR: now also U6.56 (IOB_94); no longer U6.63 (IOB_103_CBSEL0)
- net VUART_DTR: now also U6.60 (IOB_95); no longer U6.62 (IOB_102)
- net VUART_RTS: now also U6.62 (IOB_102); no longer U6.60 (IOB_95)
- net VUART_Rx: now also U6.64 (IOB_104_CBSEL1); no longer U6.55 (IOB_91)
- net VUART_Tx: now also U6.63 (IOB_103_CBSEL0); no longer U6.56 (IOB_94)
- net at U6.49 (IOB_81_GBIN5): now also JP1.2 (B); no longer Y2.3 (OUTPUT)
- net at U6.129 (IOT_198_GBIN0): now also JP2.2 (B); no longer JP1.2 (B)
- new net 100MHz_CLK: JP2.1 (A), Y2.3 (OUTPUT)
Other:
- moved on the sheet: C33, C34, C35, C36, C37, C38, C39, C40, C41, C42, C43, C44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
