File: project/azukar-fpga.kicad_pcb (KiCad board)
At the start: 2 copper layers, 100 x 75 mm, 168 parts, among them J1 USB_C_Receptacle_USB2.0_16P, P1 Conector 2x10, P2 Conector 2x10, P3 Conector 2x10, P4 Conector 2x10, SW1 SW_Push, SW2 SW_Push, SW3 SW_Push, SW4 SW_Push, SW5 SW_Push, SW6 SW_Push, SW7 SW_Push, SW8 SW_Push, U1 TLV76133DCYR, U2 TLV76112DCYR, U3 USBLC6-2SC6, U4 FT2232HL, U5 M93C66, U6 ICE40HX4K-TQ144, U7 W25X40CLSN, Y1 ECS-3225MV-120-CN-TR, Y2 ECS-3225MVQ-1000-CN-TR

Commit message: Archivos a prod en 2026, pinout placa, incoming datasheets
Parts:
- moved C30 0.07 mm to (158.8, 116.0)
- moved C42 0.07 mm to (158.8, 113.6)
